File: controller/relay.kicad_sch (KiCad schematic)
At the start: 0 parts

Commit message: vcc output vin npn collector amp
Parts:
- added D1: 1N4007, Diode_THT:D_DO-41_SOD81_P10.16mm_Horizontal, symbol Diode:1N4007
- added K1: Relay_DPDT, symbol Relay:Relay_DPDT
- added M1: Motor_DC, symbol Motor:Motor_DC
- added SW1, SW2: SW_SPST, symbol Switch:SW_SPST
Connections:
- new net: D1.1 (K), K1.12, K1.24, K1.A1, SW1.2 (B)
- new net: D1.2 (A), K1.14, K1.22, SW2.1 (A)
- new net: K1.21, M1.1 (+)
- new net: K1.11, M1.2 (-)
- new net +12V: SW1.1 (A)
- new net GND: K1.A2, SW2.2 (B)
Other:
- note added: "12V"
